Commit message: works

File: sr_ur_launch/description/ur10_robot.urdf.xacro (robot description, xacro)
@@ -7,9 +7,9 @@
   <xacro:include filename="$(find ur_description)/urdf/ur10.urdf.xacro" />
   <!-- arm -->
-  <xacro:ur10_robot prefix="ra" joint_limited="false"/>
+  <xacro:ur10_robot prefix="ra_" joint_limited="false"/>
   <link name="world" />
   <joint name="world_joint" type="fixed">
     <parent link="world" />
-    <child link = "base_link" />
+    <child link = "ra_base_link" />
     <origin xyz="0.0 0.0 0.0" rpy="0.0 0.0 0.0" />
   </joint>
