Commit message: corrected left arm prefix

File: sr_ur_launch/description/ur10_left_robot.urdf.xacro (robot description, xacro)
@@ -5,9 +5,9 @@
   <xacro:include filename="$(find ur_description)/urdf/ur10.urdf.xacro" />
   <!-- arm -->
-  <xacro:ur10_robot prefix="ra_" joint_limited="false"/>
+  <xacro:ur10_robot prefix="la_" joint_limited="false"/>
   <link name="world" />
   <joint name="world_joint" type="fixed">
     <parent link="world" />
-    <child link = "ra_base_link" />
+    <child link = "la_base_link" />
     <origin xyz="0.0 0.0 0.0" rpy="0.0 0.0 0.0" />
   </joint>

Commit message: corrected xml formatting

File: sr_ur_launch/description/ur10_left_robot.urdf.xacro (robot description, xacro)
@@ -6,8 +6,8 @@
   <!-- arm -->
   <xacro:ur10_robot prefix="la_" joint_limited="false"/>
-  <link name="world" />
+  <link name="world"/>
   <joint name="world_joint" type="fixed">
     <parent link="world" />
-    <child link = "la_base_link" />
+    <child link="la_base_link" />
     <origin xyz="0.0 0.0 0.0" rpy="0.0 0.0 0.0" />
   </joint>

File: sr_ur_launch/description/ur10_right_robot.urdf.xacro (robot description, xacro)
@@ -6,8 +6,8 @@
   <!-- arm -->
   <xacro:ur10_robot prefix="ra_" joint_limited="false"/>
-  <link name="world" />
+  <link name="world"/>
   <joint name="world_joint" type="fixed">
     <parent link="world" />
-    <child link = "ra_base_link" />
+    <child link="ra_base_link" />
     <origin xyz="0.0 0.0 0.0" rpy="0.0 0.0 0.0" />
   </joint>
